File: PCB + ArduinoCODE/hyperloop_senior-design.kicad_pcb (KiCad board)
At the start: 2 copper layers, 138.7 x 48.8 mm, 34 parts, among them J1 Screw_Terminal_01x02, J2 Screw_Terminal_01x02, SW1 SW_Push, SW2 SW_Push, U1 RN-2407S, U2 LM2937IMPX-15/NOPB, U3 L298N

Commit message: mohamed changes -v3
Parts:
- SW1, SW2: value SW_Push -> (none)
Other:
- board text added: "hyperloop_senior-design_v00"
- board text removed: "Ben Hamilton Mohamed Mahmoud Liam Waghorn"
Changed lines of the file:
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@@
     (area 31.420999 96.444999 170.255001 145.363001)
     (thickness 1.6)
-    (drawings 16)
+    (drawings 15)
     (tracks 297)
     (zones 0)
@@
     (aux_axis_origin 0 0)
     (grid_origin 75.438 131.318)
-    (visible_elements FFFFFF7F)
+    (visible_elements 7FFFFFFF)
     (pcbplotparams
       (layerselection 0x00030_80000001)
@@
       (effects (font (size 1 1) (thickness 0.15)))
     )
-    (fp_text value SW_Push (at 6.62 9.93) (layer F.Fab)
+    (fp_text value "" (at 6.62 9.93) (layer F.Fab)
       (effects (font (size 1 1) (thickness 0.15)))
     )
@@
       (effects (font (size 1 1) (thickness 0.15)))
     )
-    (fp_text value SW_Push (at 6.62 9.93) (layer F.Fab)
+    (fp_text value "" (at 6.62 9.93) (layer F.Fab)
       (effects (font (size 1 1) (thickness 0.15)))
     )
@@
     )
   )
-  (gr_line (start 101.854 141.986) (end 97.282 141.986) (angle 90) (layer F.SilkS) (width 0.2))
-  (gr_line (start 101.854 134.874) (end 101.854 141.986) (angle 90) (layer F.SilkS) (width 0.2))
-  (gr_line (start 97.282 134.874) (end 101.854 134.874) (angle 90) (layer F.SilkS) (width 0.2))
-  (gr_text "Ben Hamilton\nMohamed Mahmoud\nLiam Waghorn" (at 78.994 138.43) (layer F.SilkS)
-    (effects (font (size 1.5 1.5) (thickness 0.3)) (justify left))
-  )
-  (gr_line (start 78.486 141.986) (end 78.486 141.478) (angle 90) (layer F.SilkS) (width 0.2))
-  (gr_line (start 97.282 141.986) (end 78.486 141.986) (angle 90) (layer F.SilkS) (width 0.2))
-  (gr_line (start 78.486 134.874) (end 97.282 134.874) (angle 90) (layer F.SilkS) (width 0.2))
-  (gr_line (start 78.486 141.986) (end 78.486 134.874) (angle 90) (layer F.SilkS) (width 0.2))
+  (gr_text CCW (at 43.942 143.002) (layer F.SilkS)
+    (effects (font (size 1.5 1.5) (thickness 0.3)))
+  )
+  (gr_text "CW\n" (at 62.738 143.002) (layer F.SilkS)
+    (effects (font (size 1.5 1.5) (thickness 0.3)))
+  )
+  (gr_line (start 73.406 136.398) (end 107.95 136.398) (angle 90) (layer F.SilkS) (width 0.2))
+  (gr_line (start 73.406 143.002) (end 73.406 136.398) (angle 90) (layer F.SilkS) (width 0.2))
+  (gr_line (start 107.95 143.002) (end 73.406 143.002) (angle 90) (layer F.SilkS) (width 0.2))
+  (gr_line (start 107.95 136.398) (end 107.95 143.002) (angle 90) (layer F.SilkS) (width 0.2))
+  (gr_text hyperloop_senior-design_v00 (at 90.678 137.922) (layer F.SilkS)
+    (effects (font (size 1.5 1.5) (thickness 0.3)))
+  )
   (gr_text "IDLE\n" (at 100.33 128.27 90) (layer F.SilkS)
     (effects (font (size 1.5 1.5) (thickness 0.3)))
